Commit message: Base scenarios added

File: urdf/pioneer3at_aruco.urdf (robot description, URDF)
Before this commit: robot pioneer3at, 20 links, 19 joints
Links:
- link aruco_left: geometry visual mesh filename=package://tasks_distribution/meshes/aruco_1.dae
- link aruco_right: geometry visual mesh filename=package://tasks_distribution/meshes/aruco_2.dae
